File: hardware/Bias_PS.sch (KiCad schematic (older format))
At the start: 44 parts

Commit message: Adding ULX3S connections
Parts:
- removed C?: N.C., EEZ DIB DCM220 r2B7:C0805, symbol EEZ_DIB_DCM220_r2B7-eagle-import:C-EUC0805
- removed C?: 2u2, EEZ DIB DCM220 r2B7:C1206, symbol EEZ_DIB_DCM220_r2B7-eagle-import:C-EUC1206
- removed C? (x3): 10n/200V, EEZ DIB DCM220 r2B7:C1206, symbol EEZ_DIB_DCM220_r2B7-eagle-import:C-EUC1206
- removed C?: 10n, EEZ DIB DCM220 r2B7:C0805, symbol EEZ_DIB_DCM220_r2B7-eagle-import:C-EUC0805
- removed IC?: LP2985-33DBVR, EEZ DIB DCM220 r2B7:SOT95P270X145-5N, symbol EEZ_DIB_DCM220_r2B7-eagle-import:LP2985
- removed J?: 4907, EEZ DIB DCM220 r2B7:PCB_TAB-4907, symbol EEZ_DIB_DCM220_r2B7-eagle-import:PCB_TAB-4907
- removed L? (x2): RN112-4-02-0M7, EEZ DIB DCM220 r2B7:RN112, symbol EEZ_DIB_DCM220_r2B7-eagle-import:RN112
- removed R?: N.C., EEZ DIB DCM220 r2B7:R2512, symbol EEZ_DIB_DCM220_r2B7-eagle-import:R-EU_R2512
- removed X? (x2): 39-30-1020, EEZ DIB DCM220 r2B7:MINIFIT_39301020, symbol EEZ_DIB_DCM220_r2B7-eagle-import:MINIFIT_39301020
- removed ZD?: SMAJ51A, EEZ DIB DCM220 r2B7:DO214AA, symbol EEZ_DIB_DCM220_r2B7-eagle-import:P6SMB68A
- added C? (x3): 4.7uF/10V, symbol antena:C
- added C?: 1uF/10V, symbol antena:C
- added C?: 4.7V/10V, symbol antena:C
- added C?: 2.2uF/10V, symbol antena:C
- added R?: 494K, symbol antena:R
- added R?: 1.37M, symbol antena:R
- added R?: 100R 1/4W, symbol antena:R
- added R?: 1R, symbol antena:R
- added U?: LM27761, Package_SON:WSON-8-1EP_2x2mm_P0.5mm_EP0.9x1.6mm, symbol Regulator_SwitchedCapacitor:LM27761
- C? (x2): symbol EEZ_DIB_DCM220_r2B7-eagle-import:C-EUC0603 -> LCD_PMOD-rescue:C-EUC0603-EEZ_DIB_DCM220_r2B7-eagle-import
- C? (x2): symbol EEZ_DIB_DCM220_r2B7-eagle-import:C-EUC0805 -> LCD_PMOD-rescue:C-EUC0805-EEZ_DIB_DCM220_r2B7-eagle-import
- C? (x7): symbol EEZ_DIB_DCM220_r2B7-eagle-import:C-EUC1206 -> LCD_PMOD-rescue:C-EUC1206-EEZ_DIB_DCM220_r2B7-eagle-import
- C?: value 10n -> 3n3; symbol EEZ_DIB_DCM220_r2B7-eagle-import:C-EUC0805 -> LCD_PMOD-rescue:C-EUC0805-EEZ_DIB_DCM220_r2B7-eagle-import
- C?: value 33p -> 7p; symbol EEZ_DIB_DCM220_r2B7-eagle-import:C-EUC0603 -> LCD_PMOD-rescue:C-EUC0603-EEZ_DIB_DCM220_r2B7-eagle-import
- D? (x2): symbol EEZ_DIB_DCM220_r2B7-eagle-import:SCHOTTKYSOD123 -> LCD_PMOD-rescue:SCHOTTKYSOD123-EEZ_DIB_DCM220_r2B7-eagle-import
- IC?: symbol EEZ_DIB_DCM220_r2B7-eagle-import:AT24CXXSOIC8 -> LCD_PMOD-rescue:AT24CXXSOIC8-EEZ_DIB_DCM220_r2B7-eagle-import
- IC?: symbol EEZ_DIB_DCM220_r2B7-eagle-import:TPS54060DGQ -> LCD_PMOD-rescue:TPS54060DGQ-EEZ_DIB_DCM220_r2B7-eagle-import
- R?: value 2K2 -> 16K; symbol EEZ_DIB_DCM220_r2B7-eagle-import:R-EU_R0805 -> LCD_PMOD-rescue:R-EU_R0805-EEZ_DIB_DCM220_r2B7-eagle-import
- R? (x6): symbol EEZ_DIB_DCM220_r2B7-eagle-import:R-EU_R0805 -> LCD_PMOD-rescue:R-EU_R0805-EEZ_DIB_DCM220_r2B7-eagle-import
- R?: value 10K -> 16K; symbol EEZ_DIB_DCM220_r2B7-eagle-import:R-EU_R0805 -> LCD_PMOD-rescue:R-EU_R0805-EEZ_DIB_DCM220_r2B7-eagle-import
- R?: value 86K6 -> 130K; symbol EEZ_DIB_DCM220_r2B7-eagle-import:R-EU_R0805 -> LCD_PMOD-rescue:R-EU_R0805-EEZ_DIB_DCM220_r2B7-eagle-import
- R?: value 86K6 -> 180K; symbol EEZ_DIB_DCM220_r2B7-eagle-import:R-EU_R0805 -> LCD_PMOD-rescue:R-EU_R0805-EEZ_DIB_DCM220_r2B7-eagle-import
- R?: value 47K -> 130K; symbol EEZ_DIB_DCM220_r2B7-eagle-import:R-EU_R0805 -> LCD_PMOD-rescue:R-EU_R0805-EEZ_DIB_DCM220_r2B7-eagle-import
- R?: value 330K -> 220K; symbol EEZ_DIB_DCM220_r2B7-eagle-import:R-EU_R0805 -> LCD_PMOD-rescue:R-EU_R0805-EEZ_DIB_DCM220_r2B7-eagle-import
- TR?: value SRF0703-821M -> SRF0703-820M; symbol EEZ_DIB_DCM220_r2B7-eagle-import:BOURNS_SRF0703INV -> LCD_PMOD-rescue:BOURNS_SRF0703INV-EEZ_DIB_DCM220_r2B7-eagle-import
Connections:
- net labels added: +12V, +5V, -4V5, A0, A1, A2, HVDD, HVSS, SSCL, SSDA
- net labels removed: +3V3, PE
- wire segments 158 -> 157
Other:
- note added: "+10V"
- note added: "-10V"
- note added: "UVLO off: \nUVLO on:"
- note removed: "+3V3 LDO"
- note removed: "+48V DC input"
- note removed: "DC in (max. 55 V)"
- note removed: "UVLO off: +33 V\nUVLO on: +38 V"

Commit message: Assigning footprints
Parts:
- removed C?: 10n, EEZ DIB DCM220 r2B7:C0805, symbol LCD_PMOD-rescue:C-EUC0805-EEZ_DIB_DCM220_r2B7-eagle-import
- removed C?: 330p, EEZ DIB DCM220 r2B7:C0805, symbol LCD_PMOD-rescue:C-EUC0805-EEZ_DIB_DCM220_r2B7-eagle-import
- removed C?: N.C., EEZ DIB DCM220 r2B7:C1206, symbol LCD_PMOD-rescue:C-EUC1206-EEZ_DIB_DCM220_r2B7-eagle-import
- removed C? (x3): 4u7, EEZ DIB DCM220 r2B7:C1206, symbol LCD_PMOD-rescue:C-EUC1206-EEZ_DIB_DCM220_r2B7-eagle-import
- removed C?: 100n, EEZ DIB DCM220 r2B7:C0603, symbol LCD_PMOD-rescue:C-EUC0603-EEZ_DIB_DCM220_r2B7-eagle-import
- removed C? (x3): 4.7uF/10V, symbol antena:C
- removed C?: 1uF/10V, symbol antena:C
- removed C?: 4.7V/10V, symbol antena:C
- removed C?: 2.2uF/10V, symbol antena:C
- removed C? (x2): 2u2, EEZ DIB DCM220 r2B7:C1206, symbol LCD_PMOD-rescue:C-EUC1206-EEZ_DIB_DCM220_r2B7-eagle-import
- removed C?: 22u, EEZ DIB DCM220 r2B7:C1206, symbol LCD_PMOD-rescue:C-EUC1206-EEZ_DIB_DCM220_r2B7-eagle-import
- removed C?: 3n3, EEZ DIB DCM220 r2B7:C0805, symbol LCD_PMOD-rescue:C-EUC0805-EEZ_DIB_DCM220_r2B7-eagle-import
- removed C?: 7p, EEZ DIB DCM220 r2B7:C0603, symbol LCD_PMOD-rescue:C-EUC0603-EEZ_DIB_DCM220_r2B7-eagle-import
- removed D? (x2): SKL16, EEZ DIB DCM220 r2B7:SOD123, symbol LCD_PMOD-rescue:SCHOTTKYSOD123-EEZ_DIB_DCM220_r2B7-eagle-import
- removed IC?: TPS54060DGQ, EEZ DIB DCM220 r2B7:SOP50P490X110-11N, symbol LCD_PMOD-rescue:TPS54060DGQ-EEZ_DIB_DCM220_r2B7-eagle-import
- removed R? (x2): 16K, EEZ DIB DCM220 r2B7:R0805, symbol LCD_PMOD-rescue:R-EU_R0805-EEZ_DIB_DCM220_r2B7-eagle-import
- removed R? (x3): 10R, EEZ DIB DCM220 r2B7:R0805, symbol LCD_PMOD-rescue:R-EU_R0805-EEZ_DIB_DCM220_r2B7-eagle-import
- removed R? (x2): 130K, EEZ DIB DCM220 r2B7:R0805, symbol LCD_PMOD-rescue:R-EU_R0805-EEZ_DIB_DCM220_r2B7-eagle-import
- removed R?: 494K, symbol antena:R
- removed R?: 1.37M, symbol antena:R
- removed R?: 100R 1/4W, symbol antena:R
- removed R?: 1R, symbol antena:R
- removed R?: 180K, EEZ DIB DCM220 r2B7:R0805, symbol LCD_PMOD-rescue:R-EU_R0805-EEZ_DIB_DCM220_r2B7-eagle-import
- removed R?: 220K, EEZ DIB DCM220 r2B7:R0805, symbol LCD_PMOD-rescue:R-EU_R0805-EEZ_DIB_DCM220_r2B7-eagle-import
- removed TR?: SRF0703-820M, EEZ DIB DCM220 r2B7:SRF0703, symbol LCD_PMOD-rescue:BOURNS_SRF0703INV-EEZ_DIB_DCM220_r2B7-eagle-import
- removed U?: LM27761, Package_SON:WSON-8-1EP_2x2mm_P0.5mm_EP0.9x1.6mm, symbol Regulator_SwitchedCapacitor:LM27761
- added J8: TBA1E, Connector_PinHeader_2.54mm:PinHeader_1x06_P2.54mm_Vertical, symbol Connector_Generic:Conn_01x06
- C73: renamed from C?; footprint EEZ DIB DCM220 r2B7:C0603 -> Capacitor_SMD:C_0603_1608Metric
- IC6: renamed from IC?; footprint EEZ DIB DCM220 r2B7:SOIC127P600X173-8N -> OPA2211:SOIC127P600X170-9N
- R50, R51, R52: renamed from R?; footprint EEZ DIB DCM220 r2B7:R0805 -> Capacitor_SMD:C_0805_2012Metric
Connections:
- net GNDIO is gone; now on net GND: C73.1, IC6.4 (GND), IC6.7 (WP)
- net +12V: now also J8.1 (Pin_1)
- net GND: now also J8.2 (Pin_2)
- net V+ renamed 3V3
- new net HVDD: J8.6 (Pin_6)
- new net HVSS: J8.4 (Pin_4)
Other:
- note added: "+5V"
- note added: "-5V"
- note removed: "+0.8 V"
- note removed: "+10V"
- note removed: "-10V"
- note removed: "Bias power supply"
- note removed: "UVLO off: \nUVLO on:"

Commit message: Adding last known changes to shematics
Parts:
- removed C73: 100n, Capacitor_SMD:C_0603_1608Metric, symbol LCD_PMOD-rescue:C-EUC0603-EEZ_DIB_DCM220_r2B7-eagle-import
- removed IC6: M24C32-WMN6P, OPA2211:SOIC127P600X170-9N, symbol LCD_PMOD-rescue:AT24CXXSOIC8-EEZ_DIB_DCM220_r2B7-eagle-import
- removed J8: TBA1E, Connector_PinHeader_2.54mm:PinHeader_1x06_P2.54mm_Vertical, symbol Connector_Generic:Conn_01x06
- removed R50, R51, R52: 10K, Capacitor_SMD:C_0805_2012Metric, symbol LCD_PMOD-rescue:R-EU_R0805-EEZ_DIB_DCM220_r2B7-eagle-import
Other:
- note removed: "+5V"
- note removed: "-5V"
- note removed: "I2C Module ID EEPROM"
Changed lines of the file:
@@
 Comment4 ""
 $EndDescr
-Wire Wire Line
-	2900 6100 3200 6100
-Wire Wire Line
-	3200 6100 3200 6900
-Wire Wire Line
-	3200 6900 3200 7200
-Wire Wire Line
-	3200 7200 2900 7200
-Text Label 1300 6900 0    50   ~ 0
-DIB_A0
-Connection ~ 3200 6900
-Wire Wire Line
-	2900 6200 3100 6200
-Wire Wire Line
-	3100 6200 3100 6800
-Wire Wire Line
-	3100 6800 3100 7100
-Wire Wire Line
-	3100 7100 2900 7100
-Text Label 1300 6800 0    50   ~ 0
-DIB_A1
-Connection ~ 3100 6800
-Wire Wire Line
-	2900 6300 3000 6300
-Wire Wire Line
-	3000 6300 3000 6700
-Wire Wire Line
-	3000 6700 3000 7000
-Wire Wire Line
-	3000 7000 2900 7000
-Text Label 1300 6700 0    50   ~ 0
-DIB_A2
-Connection ~ 3000 6700
-Text Label 1300 5900 0    50   ~ 0
-DIB_SCL
-Text Label 1300 6000 0    50   ~ 0
-DIB_SDA
-Wire Wire Line
-	1900 6100 1800 6100
-Wire Wire Line
-	1800 6100 1800 6300
-Wire Wire Line
-	1800 6300 1900 6300
-Wire Wire Line
-	1800 6400 1800 6300
-Connection ~ 1800 6300
-Text Label 1900 6100 0    10   ~ 0
-GNDIO
-Wire Wire Line
-	3400 5900 3500 5900
-Text Label 3400 5900 0    10   ~ 0
-GNDIO
-Wire Wire Line
-	2900 5900 3000 5900
-Wire Wire Line
-	3100 5900 3000 5900
-Connection ~ 3000 5900
-Text Label 2900 5900 0    10   ~ 0
-V+
-Wire Wire Line
-	2500 7000 2300 7000
-Wire Wire Line
-	2300 7000 2300 7100
-Wire Wire Line
-	2300 7100 2300 7200
-Wire Wire Line
-	2300 7200 2500 7200
-Wire Wire Line
-	2500 7100 2300 7100
-Connection ~ 2300 7100
-Connection ~ 2300 7000
-Text Label 2500 7000 0    10   ~ 0
-V+
-$Comp
-L LCD_PMOD-rescue:C-EUC0603-EEZ_DIB_DCM220_r2B7-eagle-import C?
-U 1 0 1FF5D5AC1D7B263C
-P 3300 5900
-AR Path="/1FF5D5AC1D7B263C" Ref="C?"  Part="1"
-AR Path="/5E155363/1FF5D5AC1D7B263C" Ref="C?"  Part="1"
-AR Path="/5E500AA4/1FF5D5AC1D7B263C" Ref="C73"  Part="1"
-F 0 "C73" V 3285 5885 59  0000 L BNN
-F 1 "100n" V 3385 5885 59  0000 L BNN
-F 2 "Capacitor_SMD:C_0603_1608Metric" H 3300 5900 50  0001 C CNN
-F 3 "" H 3300 5900 50  0001 C CNN
-	1    3300 5900
-	0    1    1    0
-$EndComp
-$Comp
-L LCD_PMOD-rescue:R-EU_R0805-EEZ_DIB_DCM220_r2B7-eagle-import R?
-U 1 0 1F0C43AD49162B56
-P 2700 7000
-AR Path="/1F0C43AD49162B56" Ref="R?"  Part="1"
-AR Path="/5E155363/1F0C43AD49162B56" Ref="R?"  Part="1"
-AR Path="/5E500AA4/1F0C43AD49162B56" Ref="R50"  Part="1"
-F 0 "R50" H 2800 6909 59  0000 L BNN
-F 1 "10K" H 2575 6980 59  0000 R TNN
-F 2 "Capacitor_SMD:C_0805_2012Metric" H 2700 7000 50  0001 C CNN
-F 3 "" H 2700 7000 50  0001 C CNN
-	1    2700 7000
-	1    0    0    1
-$EndComp
-$Comp
-L LCD_PMOD-rescue:R-EU_R0805-EEZ_DIB_DCM220_r2B7-eagle-import R?
-U 1 0 A56A49D9FBBF1A7E
-P 2700 7100
-AR Path="/A56A49D9FBBF1A7E" Ref="R?"  Part="1"
-AR Path="/5E155363/A56A49D9FBBF1A7E" Ref="R?"  Part="1"
-AR Path="/5E500AA4/A56A49D9FBBF1A7E" Ref="R51"  Part="1"
-F 0 "R51" H 2800 7009 59  0000 L BNN
-F 1 "10K" H 2575 7080 59  0000 R TNN
-F 2 "Capacitor_SMD:C_0805_2012Metric" H 2700 7100 50  0001 C CNN
-F 3 "" H 2700 7100 50  0001 C CNN
-	1    2700 7100
-	1    0    0    1
-$EndComp
-$Comp
-L LCD_PMOD-rescue:R-EU_R0805-EEZ_DIB_DCM220_r2B7-eagle-import R?
-U 1 0 6482207A2BD16012
-P 2700 7200
-AR Path="/6482207A2BD16012" Ref="R?"  Part="1"
-AR Path="/5E155363/6482207A2BD16012" Ref="R?"  Part="1"
-AR Path="/5E500AA4/6482207A2BD16012" Ref="R52"  Part="1"
-F 0 "R52" H 2800 7109 59  0000 L BNN
-F 1 "10K" H 2575 7180 59  0000 R TNN
-F 2 "Capacitor_SMD:C_0805_2012Metric" H 2700 7200 50  0001 C CNN
-F 3 "" H 2700 7200 50  0001 C CNN
-	1    2700 7200
-	1    0    0    1
-$EndComp
-$Comp
-L LCD_PMOD-rescue:AT24CXXSOIC8-EEZ_DIB_DCM220_r2B7-eagle-import IC?
-U 1 0 3E9A5E0E738E3039
-P 2400 6100
-AR Path="/3E9A5E0E738E3039" Ref="IC?"  Part="1"
-AR Path="/5E155363/3E9A5E0E738E3039" Ref="IC?"  Part="1"
-AR Path="/5E500AA4/3E9A5E0E738E3039" Ref="IC6"  Part="1"
-F 0 "IC6" H 2314 6434 69  0000 L BNN
-F 1 "M24C32-WMN6P" H 1964 5683 69  0000 L BNN
-F 2 "OPA2211:SOIC127P600X170-9N" H 2400 6100 50  0001 C CNN
-F 3 "" H 2400 6100 50  0001 C CNN
-	1    2400 6100
-	1    0    0    -1
-$EndComp
-Text Notes 1100 5400 0    59   ~ 0
-I2C Module ID EEPROM
-Wire Notes Line
-	3700 7600 3700 5300
-Text GLabel 1200 6000 0    50   Input ~ 0
-SSDA
-Wire Wire Line
-	1200 6000 1900 6000
-Text GLabel 1200 5900 0    50   Input ~ 0
-SSCL
-Wire Wire Line
-	1200 5900 1900 5900
-Text GLabel 1200 6900 0    50   Input ~ 0
-A0
-Text GLabel 1200 6800 0    50   Input ~ 0
-A1
-Text GLabel 1200 6700 0    50   Input ~ 0
-A2
-Wire Wire Line
-	1200 6700 3000 6700
-Wire Wire Line
-	1200 6800 3100 6800
-Wire Wire Line
-	1200 6900 3200 6900
-Text Notes 1500 4600 0    50   ~ 0
--5V
-Text Notes 1500 4800 0    50   ~ 0
-+5V
-$Comp
-L Connector_Generic:Conn_01x06 J8
-U 1 1 5E7E704B
-P 2250 4450
-F 0 "J8" H 2329 4442 50  0000 L CNN
-F 1 "TBA1E" H 2329 4351 50  0000 L CNN
-F 2 "Connector_PinHeader_2.54mm:PinHeader_1x06_P2.54mm_Vertical" H 2250 4450 50  0001 C CNN
-F 3 "~" H 2250 4450 50  0001 C CNN
-	1    2250 4450
-	1    0    0    -1
-$EndComp
-Text GLabel 1950 4250 0    50   Input ~ 0
-+12V
-Text GLabel 1950 4350 0    50   Input ~ 0
-GND
-Text GLabel 1950 4550 0    50   Input ~ 0
-HVSS
-Text GLabel 1950 4750 0    50   Input ~ 0
-HVDD
-Wire Wire Line
-	1950 4250 2050 4250
-Wire Wire Line
-	1950 4350 2050 4350
-Wire Wire Line
-	1950 4550 2050 4550
-Wire Wire Line
-	1950 4750 2050 4750
-Text GLabel 3500 6100 3    50   Input ~ 0
-GND
-Wire Wire Line
-	3500 5900 3500 6100
-Text GLabel 1800 6400 3    50   Input ~ 0
-GND
-Text GLabel 3000 5700 1    50   Input ~ 0
-3V3
-Text GLabel 2100 7000 0    50   Input ~ 0
-3V3
-Wire Wire Line
-	3000 5700 3000 5900
-Wire Wire Line
-	2100 7000 2300 7000
 $EndSCHEMATC
