File: hardware/ADC_buffer.sch (KiCad schematic (older format))
At the start: 25 parts

Commit message: Adding AMC1304 to the board
Parts:
- added IC?: TPD4E001-DRL, symbol EEZ_DIB_MCU_r1B1-eagle-import:TPD4E001-DRL
- added R?: 1K, symbol antena:R
- added U?: AMC1304L, symbol AMC1304M:AMC1304L
Connections:
- net labels added: A1_IN, AVDD, B0_IN, B1_IN
- wire segments 73 -> 88
Changed lines of the file:
@@
 Wire Wire Line
 	10350 1950 10700 1950
+$Comp
+L EEZ_DIB_MCU_r1B1-eagle-import:TPD4E001-DRL IC?
+U 1 1 5E7CC48A
+P 2250 4600
+F 0 "IC?" H 2250 5008 69  0000 C CNN
+F 1 "TPD4E001-DRL" H 2250 4888 69  0000 C CNN
+F 2 "" H 2250 4600 50  0001 C CNN
+F 3 "" H 2250 4600 50  0001 C CNN
+	1    2250 4600
+	1    0    0    -1
+$EndComp
+Text GLabel 1650 4500 0    50   Input ~ 0
+A0_IN
+Text GLabel 1650 4600 0    50   Input ~ 0
+A1_IN
+Text GLabel 1650 4700 0    50   Input ~ 0
+B0_IN
+Text GLabel 1650 4800 0    50   Input ~ 0
+B1_IN
+Wire Wire Line
+	1650 4500 1750 4500
+Wire Wire Line
+	1650 4600 1750 4600
+Wire Wire Line
+	1650 4700 1750 4700
+Wire Wire Line
+	1650 4800 1750 4800
+Text GLabel 2900 4800 2    50   Input ~ 0
+AGND
+Text GLabel 2900 4500 2    50   Input ~ 0
+AVDD
+Wire Wire Line
+	2750 4500 2900 4500
+Wire Wire Line
+	2750 4800 2900 4800
+Text GLabel 9200 1250 1    50   Input ~ 0
+AVDD
+Wire Wire Line
+	9200 1250 9200 1450
+Wire Wire Line
+	9200 1450 9000 1450
+Text GLabel 9200 2300 3    50   Input ~ 0
+AGND
+Wire Wire Line
+	9000 2150 9200 2150
+Wire Wire Line
+	9200 2150 9200 2300
+$Comp
+L antena:R R?
+U 1 1 5E7E0234
+P 7300 1300
+F 0 "R?" V 7507 1300 50  0000 C CNN
+F 1 "1K" V 7416 1300 50  0000 C CNN
+F 2 "" V 7230 1300 50  0001 C CNN
+F 3 "~" H 7300 1300 50  0001 C CNN
+	1    7300 1300
+	0    -1   -1   0
+$EndComp
+Wire Wire Line
+	7450 1300 7900 1300
+Wire Wire Line
+	7900 1300 7900 1450
+Wire Wire Line
+	7900 1450 8000 1450
+Text GLabel 7000 1150 1    50   Input ~ 0
+AVDD
+Wire Wire Line
+	7000 1150 7000 1300
+Wire Wire Line
+	7000 1300 7150 1300
+$Comp
+L AMC1304M:AMC1304L U?
+U 1 1 5E2A7202
+P 7850 4550
+F 0 "U?" H 7850 5317 50  0000 C CNN
+F 1 "AMC1304L" H 7850 5226 50  0000 C CNN
+F 2 "" H 7850 4550 50  0001 C CNN
+F 3 "http://www.ti.com/lit/ds/symlink/amc1304m05.pdf" H 7850 4550 50  0001 C CNN
+	1    7850 4550
+	1    0    0    -1
+$EndComp
 $EndSCHEMATC

Commit message: Adding ULX3S connections
Parts:
- removed U?: AMC1304L, symbol AMC1304M:AMC1304L
- added C?: 1n, symbol antena:C
- added C?: 470p, symbol antena:C
- added C?: 22nF, symbol antena:C
- added C? (x2): 270pF, symbol antena:C
- added IC?: TPD4E001-DRL, symbol EEZ_DIB_MCU_r1B1-eagle-import:TPD4E001-DRL
- added R? (x2): 300R, symbol antena:R
- added R? (x4): 1K2, symbol antena:R
- added R? (x2): 5R, symbol antena:R
- added R? (x2): 10R, symbol antena:R
- added R?: 1K, symbol antena:R
- added U?: THS4551IDGKT, SOP65P490X110-8N, symbol THS4551IDGKT:THS4551IDGKT
Connections:
- net labels added: ADC_C0, ADC_C1, C0_IN, C1_IN
- net labels removed: A1N_IN, A1P_IN
- wire segments 88 -> 146

Commit message: Assigning footprints
Parts:
- C60, C61, C62, C63, C64, C65, C66, C67, C68, C69, C70, C71, C72: renamed from C?; footprint (none) -> Capacitor_SMD:C_0603_1608Metric
- IC4, IC5: renamed from IC?; footprint (none) -> Package_TO_SOT_SMD:SOT-23-6
- J7: renamed from J?; footprint (none) -> Connector_PinHeader_2.54mm:PinHeader_1x03_P2.54mm_Vertical
- R24, R25, R26, R27, R28, R29, R30, R31, R32, R33, R34, R35, R36, R37, R38, R39, R40, R41, R42, R43, R44, R45, R46, R47, R48, R49: renamed from R?; footprint (none) -> Resistor_SMD:R_0805_2012Metric
- U6: renamed from U?; footprint SOIC127P600X175-8N -> EEZ DIB MCU r1B1:SOIC127P600X173-8N
- U7, U8: renamed from U?; footprint SOP65P490X110-8N -> Package_SO:VSSOP-8_3.0x3.0mm_P0.65mm

Commit message: Adding chip power down fix - removing ADS8556 chip
Parts:
- added D2, D3, D4: D_TVS, Diode_SMD:D_SOD-523, symbol antena:D_TVS
- added R53: 1K, Resistor_SMD:R_1206_3216Metric, symbol antena:R
- R30, R31: footprint Resistor_SMD:R_0805_2012Metric -> Resistor_SMD:R_1206_3216Metric
Connections:
- net A0_IN: now also R53.2; no longer J7.2 (Pin_2), R24.2
- net A1_IN: now also D2.2 (A2), D3.2 (A2), D4.2 (A2)
- net at C64.2, R30.1, R36.2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: now also D3.1 (A1)
- net at C64.1, R31.1, R37.2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: now also D4.1 (A1)
- new net: D2.1 (A1), J7.2 (Pin_2), R24.2, R53.1
Other:
- moved on the sheet: R30, R31
Changed lines of the file:
@@
 Text GLabel 5150 1450 2    50   Input ~ 0
 ADC_A0
-Text GLabel 1150 1650 0    50   Input ~ 0
+Text GLabel 750  1650 0    50   Input ~ 0
 A0_IN
 Text GLabel 1800 2150 3    50   Input ~ 0
@@
 Connection ~ 1800 1650
 Wire Wire Line
-	1150 1650 1250 1650
-Wire Wire Line
 	1250 1650 1250 1000
 Wire Wire Line
@@
 L antena:R R30
 U 1 1 5E7A0576
-P 6400 1650
-F 0 "R30" V 6193 1650 50  0000 C CNN
-F 1 "1K2" V 6284 1650 50  0000 C CNN
-F 2 "Resistor_SMD:R_0805_2012Metric" V 6330 1650 50  0001 C CNN
-F 3 "~" H 6400 1650 50  0001 C CNN
-	1    6400 1650
+P 6000 1650
+F 0 "R30" V 5793 1650 50  0000 C CNN
+F 1 "1K2" V 5884 1650 50  0000 C CNN
+F 2 "Resistor_SMD:R_1206_3216Metric" V 5930 1650 50  0001 C CNN
+F 3 "~" H 6000 1650 50  0001 C CNN
+	1    6000 1650
 	0    1    1    0
 $EndComp
@@
 L antena:R R31
 U 1 1 5E7A05CA
-P 6400 1950
-F 0 "R31" V 6193 1950 50  0000 C CNN
-F 1 "1K2" V 6284 1950 50  0000 C CNN
-F 2 "Resistor_SMD:R_0805_2012Metric" V 6330 1950 50  0001 C CNN
-F 3 "~" H 6400 1950 50  0001 C CNN
-	1    6400 1950
-	0    1    1    0
-$EndComp
-Wire Wire Line
-	6550 1650 6800 1650
+P 6000 1950
+F 0 "R31" V 5793 1950 50  0000 C CNN
+F 1 "1K2" V 5884 1950 50  0000 C CNN
+F 2 "Resistor_SMD:R_1206_3216Metric" V 5930 1950 50  0001 C CNN
+F 3 "~" H 6000 1950 50  0001 C CNN
+	1    6000 1950
+	0    1    1    0
+$EndComp
 Connection ~ 6800 1650
-Wire Wire Line
-	6550 1950 6800 1950
 Connection ~ 6800 1950
-Text GLabel 6050 1650 0    50   Input ~ 0
+Text GLabel 5650 1650 0    50   Input ~ 0
 B0_IN
-Text GLabel 6050 1950 0    50   Input ~ 0
+Text GLabel 5650 1950 0    50   Input ~ 0
 B1_IN
 Wire Wire Line
-	6050 1650 6250 1650
-Wire Wire Line
-	6050 1950 6250 1950
+	5650 1650 5850 1650
+Wire Wire Line
+	5650 1950 5850 1950
 $Comp
 L antena:R R44
@@
 A1_IN
 Wire Wire Line
-	1150 2000 1350 2000
+	1150 2000 1250 2000
 $Comp
 L THS4551IDGKT:THS4551IDGKT U7
@@
 Wire Wire Line
 	2750 5800 2850 5800
+$Comp
+L antena:D_TVS D2
+U 1 1 5E30CD18
+P 1250 1800
+F 0 "D2" V 1204 1879 50  0000 L CNN
+F 1 "D_TVS" V 1295 1879 50  0000 L CNN
+F 2 "Diode_SMD:D_SOD-523" H 1250 1800 50  0001 C CNN
+F 3 "~" H 1250 1800 50  0001 C CNN
+	1    1250 1800
+	0    1    1    0
+$EndComp
+Wire Wire Line
+	1250 1950 1250 2000
+Connection ~ 1250 2000
+Wire Wire Line
+	1250 2000 1350 2000
+$Comp
+L antena:D_TVS D3
+U 1 1 5E3140CA
+P 6250 2200
+F 0 "D3" V 6204 2279 50  0000 L CNN
+F 1 "D_TVS" V 6295 2279 50  0000 L CNN
+F 2 "Diode_SMD:D_SOD-523" H 6250 2200 50  0001 C CNN
+F 3 "~" H 6250 2200 50  0001 C CNN
+	1    6250 2200
+	0    1    1    0
+$EndComp
+$Comp
+L antena:R R53
+U 1 1 5E314E13
+P 950 1650
+F 0 "R53" V 743 1650 50  0000 C CNN
+F 1 "1K" V 834 1650 50  0000 C CNN
+F 2 "Resistor_SMD:R_1206_3216Metric" V 880 1650 50  0001 C CNN
+F 3 "~" H 950 1650 50  0001 C CNN
+	1    950  1650
+	0    1    1    0
+$EndComp
+Wire Wire Line
+	750  1650 800  1650
+Wire Wire Line
+	1100 1650 1250 1650
+$Comp
+L antena:D_TVS D4
+U 1 1 5E3226C0
+P 6600 2200
+F 0 "D4" V 6554 2279 50  0000 L CNN
+F 1 "D_TVS" V 6645 2279 50  0000 L CNN
+F 2 "Diode_SMD:D_SOD-523" H 6600 2200 50  0001 C CNN
+F 3 "~" H 6600 2200 50  0001 C CNN
+	1    6600 2200
+	0    1    1    0
+$EndComp
+Wire Wire Line
+	6150 1650 6250 1650
+Wire Wire Line
+	6150 1950 6600 1950
+Wire Wire Line
+	6250 2050 6250 1650
+Connection ~ 6250 1650
+Wire Wire Line
+	6250 1650 6800 1650
+Wire Wire Line
+	6600 2050 6600 1950
+Connection ~ 6600 1950
+Wire Wire Line
+	6600 1950 6800 1950
+Text GLabel 6250 2450 3    50   Input ~ 0
+AGND
+Text GLabel 6600 2450 3    50   Input ~ 0
+AGND
+Wire Wire Line
+	6600 2350 6600 2450
+Wire Wire Line
+	6250 2350 6250 2450
 $EndSCHEMATC

Commit message: Adding last known changes to shematics
Parts:
- removed IC4, IC5: TPD4E001-DRL, Package_TO_SOT_SMD:SOT-23-6, symbol EEZ_DIB_MCU_r1B1-eagle-import:TPD4E001-DRL
- added C? (x2): 100n, Capacitor_SMD:C_0603_1608Metric, symbol antena:C
- added C?: 1nF, Capacitor_SMD:C_0603_1608Metric, symbol antena:C
- added C? (x2): CP, symbol antena:CP
- added D? (x3): D_TVS, Diode_SMD:D_SOD-523, symbol antena:D_TVS
- added J?: TBA1E, Connector_PinHeader_2.54mm:PinHeader_1x06_P2.54mm_Vertical, symbol Connector_Generic:Conn_01x06
- added R? (x3): 1K, Resistor_SMD:R_1206_3216Metric, symbol antena:R
Connections:
- net A0_IN is gone; now on net A1_IN: R53.2
- net A1_IN: no longer C60.2, C62.2, D2.2 (A2), D3.2 (A2), D4.2 (A2), R25.1, U7.6 (VS-), U8.6 (VS-)
- net HVDD: now also C?.1, C?.1, J?.6 (Pin_6)
- net HVSS: now also C?.1, C?.1, J?.4 (Pin_4)
- net at C63.2, R28.1, R33.2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: now also D?.1 (A1)
- net at C63.1, R29.1, R34.2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: now also D?.1 (A1)
- net ADC_A0 renamed ADC_A1P
- net ADC_B0 renamed ADC_A2P
- net ADC_B1 renamed ADC_A3P
- net ADC_C0 renamed ADC_A4P
- net ADC_C1 renamed ADC_A5P
- net B0_IN renamed A2_IN
- net B1_IN renamed A3_IN
- net C0_IN renamed A4_IN
- net C1_IN renamed A5_IN
- new net: D?.1 (A1), R?.1, R?.2
- new net +12V: J?.1 (Pin_1)
- new net A6_IN: R?.2
- new net ADC_A1GND: C62.2
- new net ADC_A6GND: C?.2, R?.1
- new net ADC_A6P: C?.1, R?.1
- new net AGND: C60.2, C?.2, C?.2, C?.2, C?.2, D2.2 (A2), D3.2 (A2), D4.2 (A2), D?.2 (A2), D?.2 (A2), D?.2 (A2), R25.1, R?.2, U7.6 (VS-), U8.6 (VS-)
- new net GND: J?.2 (Pin_2)
Other:
- note added: "+5V"
- note added: "-5V"
- note added: "TBA1E"
- moved on the sheet: C63, C64, C65, C66, C67, C68, C69, C70, C71, C72, D3, D4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

Commit message: Renaming wires
Parts:
- added R?: 49R9, Resistor_SMD:R_0805_2012Metric, symbol antena:R
Connections:
- net ADC_A1GND: now also C60.2, R?.1
- net AGND: now also R?.2; no longer C60.2
Other:
- note added: "ADC_A1N bih dovukao na C60 \ni spojio ih s 49R9 na AGND od D2\ntako da imamo sli?nu stvar kao za ADC_A6"
Changed lines of the file:
@@
 Text GLabel 750  1650 0    50   Input ~ 0
 A1_IN
-Text GLabel 1800 2150 3    50   Input ~ 0
-AGND
 Wire Wire Line
 	2400 1750 2050 1750
@@
 	2350 1450 2400 1450
 Wire Wire Line
-	1800 2050 1800 2150
-Wire Wire Line
 	1800 1750 1800 1650
 Wire Wire Line
@@
 Wire Wire Line
 	7250 1450 7400 1450
-Text GLabel 1250 2100 3    50   Input ~ 0
-AGND
 $Comp
 L THS4551IDGKT:THS4551IDGKT U7
@@
 Wire Wire Line
 	6500 2500 6500 2600
-Wire Wire Line
-	1250 1950 1250 2100
 $Comp
 L antena:D_TVS D?
@@
 Wire Notes Line
 	500  3900 500  500
+Text Notes 2550 3500 0    50   ~ 0
+ADC_A1N bih dovukao na C60 \ni spojio ih s 49R9 na AGND od D2\ntako da imamo sli?nu stvar kao za ADC_A6
+$Comp
+L antena:R R?
+U 1 1 5E905844
+P 1500 2200
+F 0 "R?" V 1293 2200 50  0000 C CNN
+F 1 "49R9" V 1384 2200 50  0000 C CNN
+F 2 "Resistor_SMD:R_0805_2012Metric" V 1430 2200 50  0001 C CNN
+F 3 "~" H 1500 2200 50  0001 C CNN
+	1    1500 2200
+	0    1    1    0
+$EndComp
+Wire Wire Line
+	1250 2200 1350 2200
+Wire Wire Line
+	1250 1950 1250 2200
+Text GLabel 1250 2350 3    50   Input ~ 0
+AGND
+Wire Wire Line
+	1800 2050 1800 2200
+Text GLabel 1800 2350 3    50   Input ~ 0
+ADC_A1GND
+Wire Wire Line
+	1650 2200 1800 2200
+Wire Wire Line
+	1800 2350 1800 2200
+Connection ~ 1800 2200
+Wire Wire Line
+	1250 2350 1250 2200
+Connection ~ 1250 2200
 $EndSCHEMATC

Commit message: Routing board
Parts:
- removed J?: TBA1E, Connector_PinHeader_2.54mm:PinHeader_1x06_P2.54mm_Vertical, symbol Connector_Generic:Conn_01x06
- added J16: TBA1E, TBA1E:TBA1E, symbol TBA1E:TBA1E
- C31: renamed from C?; footprint (none) -> Capacitor_SMD:C_0805_2012Metric
- C36: renamed from C?; footprint (none) -> Capacitor_Tantalum_SMD:CP_EIA-3528-21_Kemet-B
- J7: footprint Connector_PinHeader_2.54mm:PinHeader_1x03_P2.54mm_Vertical -> Connector_PinHeader_2.00mm:PinHeader_1x03_P2.00mm_Vertical
- R24, R28, R29, R33, R34, R36, R37: footprint Resistor_SMD:R_0805_2012Metric -> Resistor_SMD:R_1206_3216Metric
- gave numbers to parts that had none: 10
Connections:
- net +12V: now also J16.1 (+Vin_(Vcc))
- net GND: now also J16.2 (–Vin_(GND))
- net HVDD: now also J16.6 (+Vout)
- net HVSS: now also J16.4 (–Vout)
- net A2P: now reaches C64.2, D3.1 (A1), R30.1, R36.2, R40.2
- net A2N: now reaches C64.1, D4.1 (A1), R31.1, R37.2, R41.2
- net U7N: now reaches C65.1, C68.1, R34.1, U7.1 (IN-)
- net A4_out+: now reaches C67.2, R42.2, U7.4 (OUT+)
- net A4_out-: now reaches C68.2, R43.2, U7.5 (OUT-)
- net U7P: now reaches C65.2, C67.1, R33.1, U7.8 (IN+)
- net A4P: now reaches C63.2, D6.1 (A1), R28.1, R33.2, R38.2
- net A4N: now reaches C63.1, D7.1 (A1), R29.1, R34.2, R39.2
- net A4_out2+: now reaches R38.1, R42.1, R46.2
- net A4_out2-: now reaches R39.1, R43.1, R47.2
- net U8N: now reaches C66.1, C70.1, R37.1, U8.1 (IN-)
- net A2_out+: now reaches C69.2, R44.2, U8.4 (OUT+)
- net A2_out-: now reaches C70.2, R45.2, U8.5 (OUT-)
- net U8P: now reaches C66.2, C69.1, R36.1, U8.8 (IN+)
- net A2_out2+: now reaches R40.1, R44.1, R48.2
- net A2_out2-: now reaches R41.1, R45.1, R49.2
- net A2_IN renamed A2_IN_P
- net A3_IN renamed A2_IN_N
- net A4_IN renamed A4_IN_P
- net A5_IN renamed A4_IN_N
- net ADC_A2P renamed ADC_A2_OUT_P
- net ADC_A3P renamed ADC_A2_OUT_N
- net ADC_A4P renamed ADC_A4_OUT_P
- net ADC_A5P renamed ADC_A4_OUT_N
Other:
- moved on the sheet: C30, C31, C32, C36
