File: hardware/LCD_PMOD.kicad_pcb (KiCad board)
At the start: 2 copper layers, 175.3 x 95.2 mm, 174 parts, among them IC1 TPS61169DCKR, IC2 TPD4E001DRLR, IC3 AR1021-I/SS, IC4 M24C32-WMN6P, J1 20-pin power socket, J10 OS0, J11 OS1, J12 OS2, J13 PAR, J14 RANGE, J15 REF, J16 MDD01, J17 FTDI, J18 Conn_01x10, J2 VS_SCL, J3 28-pin module socket, J4 691327310016, J5 691327310016, J6 HS_SDA, J7 JMP_A0, J8 DE_IRQ, J9 DIB_V2, U1 ADS8586S, U2 REF5025AD, U3 DS90CF364AMTD, U4 DS90CF36B, U5 MC78L05_SO8, U6 THS4032ID, U7 THS4551IDGKT, U8 THS4551IDGKT, U9 MC79L05_SO8

Commit message: Adding version number
Other:
- board text added: "Ver: 0.1"
Changed lines of the file:
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@@
   (general
     (thickness 1.6)
-    (drawings 45)
+    (drawings 46)
     (tracks 4924)
     (zones 0)
@@
       (net 17 OUT-))
   )
+  (gr_text "Ver: 0.1" (at 85.59 45.27) (layer F.SilkS)
+    (effects (font (size 3 3) (thickness 0.6)))
+  )
   (gr_arc (start 59.5 124.638) (end 57.9 124.638) (angle -90) (layer Edge.Cuts) (width 1))
